Commit message: Update stretch_description.urdf

File: stretch_description/stretch_description/urdf/stretch_description.urdf (robot description, URDF)
Before this commit: robot stretch_description, 30 links, 29 joints
Links:
- link base_link: mass 1.01138852370462 -> 1.01138852370461
- link link_gripper_finger_left: mass 0.047621 -> 0.0476207785199479
- link link_gripper_finger_right: mass 0.047621 -> 0.047620778519948
- link link_gripper_fingertip_left: mass 0.0038216 -> 0.00382160686584851
- link link_gripper_fingertip_right: mass 0.0038216 -> 0.00382160881468841
- link link_left_wheel: mass 0.00356714564938457 -> 0.00356714564938459
- link link_straight_gripper: mass 0.049638 -> 0.0496384234458285
- link link_wrist_pitch: mass 0.070127 -> 0.0701267146295584
- link link_wrist_roll: mass 0.0058567 -> 0.00585666394358811
- link link_wrist_yaw: mass 0.0405398981326229 -> 0.040539898132623
- link link_wrist_yaw_bottom: mass 0.098891 -> 0.0988906816399982
Joints:
- joint joint_gripper_finger_left: axis 0 0 1 -> 0 0 -1; limit effort=0 velocity=0 -> (none); origin xyz=0.018599 0.003 0.033689 rpy=1.5708 -1.5708 0 -> xyz=0.0185992414250199 0.0029999999999975 0.0336888959851238 rpy=1.5707963267949 -1.5707963267949 0
- joint joint_gripper_finger_right: origin xyz=-0.0185992414250129 0.00300000000000195 0.0336888959851236 rpy=1.5707963267949 -1.5707963267949 0 -> xyz=-0.0185992414250104 0.00300000000000022 0.0336888959851238 rpy=1.5707963267949 1.5707963267949 0
- joint joint_gripper_fingertip_left: origin xyz=0.1906 0.006042 0 rpy=-1.5708 -4.5128E-14 -2.6011 -> xyz=0.190596948563868 -0.00604200491773282 0 rpy=1.57079632679496 4.51275387511463E-14 2.60113659715756
- joint joint_gripper_fingertip_right: origin xyz=0.190596948563868 0.00604200491758022 0 rpy=-1.57079632679483 -3.43320051448326E-14 -2.60113659715756 -> xyz=-0.190596948563868 -0.00604200491758269 0 rpy=-1.57079632679483 -3.43320051448326E-14 0.540456056432235
- joint joint_straight_gripper: origin xyz=0 0 0.0155 rpy=3.54987407349455E-30 3.24021254484265E-20 6.83173341356343E-15 -> xyz=0 0 0.0155 rpy=3.54987407349455E-30 3.24021254484265E-20 -3.14159265358979
- joint joint_wrist_roll: origin xyz=-0.0188587444076125 -0.0239999999998942 0.01955 rpy=3.14159265358979 -1.5707963267949 0 -> xyz=-0.0188587444076125 -0.0239999999998942 0.01955 rpy=3.14159265358979 1.5707963267949 0
