Commit message: docking station urdf wip

File: tool_share/stretch_docking_station_beta/stretch_description/urdf/stretch_docking_station_beta.urdf (robot description, URDF)
Before this commit: robot Stretch_RE1_docking_station_beta_URDF, 2 links, 1 joints
Links:
- link link_aruco_110mm: geometry collision mesh filename=./meshes/link_aruco_110mm.STL; visual mesh filename=./meshes/link_aruco_110mm.STL
- link link_docking_station: geometry collision mesh filename=./meshes/link_docking_station.STL; visual mesh filename=./meshes/link_docking_station.STL
