Commit message: docking station urdf beta ready

File: tool_share/stretch_docking_station_beta/stretch_docking_station_description/urdf/stretch_docking_station_description.urdf (robot description, URDF)
Before this commit: robot stretch_docking_station_description, 2 links, 1 joints
Links:
- link link_aruco_110mm: geometry collision mesh filename=./meshes/link_aruco_110mm.STL; visual mesh filename=./meshes/link_aruco_110mm.STL
- link link_docking_station: mass 1 -> None; geometry collision mesh filename=./meshes/link_docking_station.STL; visual mesh filename=./meshes/link_docking_station.STL
