Commit message: Tablet 12in urdf working in viz tool

File: tool_share_SE3/eoa_wrist_dw3_tool_tablet_12in/xacro/stretch_tool_tablet_12in.xacro (robot description, xacro)
@@ -1,48 +1,4 @@
-<?xml version="1.0" encoding="utf-8"?>
-<!-- This URDF was automatically created by SolidWorks to URDF Exporter! Originally created by Stephen Brawner (brawner@gmail.com)
-     Commit Version: 1.5.1-0-g916b5db  Build Version: 1.5.7152.31018
-     For more information, please see http://wiki.ros.org/sw_urdf_exporter -->
-<robot
-  name="stretch_description_SE3_Tablet_12in.SLDASM">
-  <link
-    name="link_wrist_roll">
-    <inertial>
-      <origin
-        xyz="0.000282866583078745 0.000557472767112321 0.0196635450474179"
-        rpy="0 0 0" />
-      <mass
-        value="0.0221916689638079" />
-      <inertia
-        ixx="2.20608319376175E-06"
-        ixy="3.01742816610977E-09"
-        ixz="-1.83537060988679E-08"
-        iyy="2.91436292743444E-06"
-        iyz="-4.55097054416199E-08"
-        izz="4.83731409646016E-06" />
-    </inertial>
-    <visual>
-      <origin
-        xyz="0 0 0"
-        rpy="0 0 0" />
-      <geometry>
-        <mesh
-          filename="package://stretch_description_SE3_Tablet_12in.SLDASM/meshes/link_wrist_roll.STL" />
-      </geometry>
-      <material
-        name="">
-        <color
-          rgba="0.898039215686275 0.917647058823529 0.929411764705882 1" />
-      </material>
-    </visual>
-    <collision>
-      <origin
-        xyz="0 0 0"
-        rpy="0 0 0" />
-      <geometry>
-        <mesh
-          filename="package://stretch_description_SE3_Tablet_12in.SLDASM/meshes/link_wrist_roll.STL" />
-      </geometry>
-    </collision>
-  </link>
+<?xml version="1.0"?>
+<robot xmlns:xacro="http://www.ros.org/wiki/xacro" name="stretch_tool_tablet_12in">
   <link
     name="link_DW3_tablet_12in">
@@ -67,5 +23,5 @@
       <geometry>
         <mesh
-          filename="package://stretch_description_SE3_Tablet_12in.SLDASM/meshes/link_DW3_tablet_12in.STL" />
+          filename="./meshes/link_DW3_tablet_12in.STL" />
       </geometry>
       <material
@@ -81,5 +37,5 @@
       <geometry>
         <mesh
-          filename="package://stretch_description_SE3_Tablet_12in.SLDASM/meshes/link_DW3_tablet_12in.STL" />
+          filename="./meshes/link_DW3_tablet_12in_collision.STL" />
       </geometry>
     </collision>
